File: Hardware/bluetoothGame.sch (KiCad schematic (older format))
At the start: 39 parts, among them J1 USB_B_Micro, Q1 UM6K33NTN, U1 LIS3DH, U2 BT840, U3 MCP73831-2-OT, Y1 32.768khz

Commit message: remake programming adapter to be much more flexable
Parts:
- D1, D2, D3, D4, D5, D6, D7, D8: symbol BudKiCadComponent:LED_Cree-PLCC4 -> bluetoothGame-rescue:LED_Cree-PLCC4-BudKiCadComponent
- D9: symbol BudKiCadComponent:D_TVS_DF5A6.8LJE -> bluetoothGame-rescue:D_TVS_DF5A6.8LJE-BudKiCadComponent
- Q1: symbol BudKiCadComponent:UM6K33NTN -> bluetoothGame-rescue:UM6K33NTN-BudKiCadComponent
- U1: symbol BudKiCadComponent:LIS3DH -> bluetoothGame-rescue:LIS3DH-BudKiCadComponent
- U2: symbol Fanstel-modules:BT840 -> bluetoothGame-rescue:BT840-Fanstel-modules
Changed lines of the file:
@@
 	15350 2250 15400 2250
 $Comp
-L BudKiCadComponent:LIS3DH U1
+L bluetoothGame-rescue:LIS3DH-BudKiCadComponent U1
 U 1 1 5C27AAD6
 P 3700 8550
@@
 $EndComp
 $Comp
-L Fanstel-modules:BT840 U2
+L bluetoothGame-rescue:BT840-Fanstel-modules U2
 U 1 1 5C2807C6
 P 10850 5650
@@
 	13300 1250 13300 1300
 $Comp
-L BudKiCadComponent:D_TVS_DF5A6.8LJE D9
+L bluetoothGame-rescue:D_TVS_DF5A6.8LJE-BudKiCadComponent D9
 U 1 1 5C29D423
 P 14700 5750
@@
 	15050 4850 15250 4850
 $Comp
-L BudKiCadComponent:LED_Cree-PLCC4 D2
+L bluetoothGame-rescue:LED_Cree-PLCC4-BudKiCadComponent D2
 U 1 1 5C2AC05D
 P 2150 2550
@@
 $EndComp
 $Comp
-L BudKiCadComponent:LED_Cree-PLCC4 D1
+L bluetoothGame-rescue:LED_Cree-PLCC4-BudKiCadComponent D1
 U 1 1 5C2AC11D
 P 2000 5450
@@
 	3650 9300 3700 9300
 $Comp
-L BudKiCadComponent:LED_Cree-PLCC4 D4
+L bluetoothGame-rescue:LED_Cree-PLCC4-BudKiCadComponent D4
 U 1 1 5C2B8818
 P 2700 2550
@@
 $EndComp
 $Comp
-L BudKiCadComponent:LED_Cree-PLCC4 D3
+L bluetoothGame-rescue:LED_Cree-PLCC4-BudKiCadComponent D3
 U 1 1 5C2B881E
 P 2550 5450
@@
 $EndComp
 $Comp
-L BudKiCadComponent:LED_Cree-PLCC4 D6
+L bluetoothGame-rescue:LED_Cree-PLCC4-BudKiCadComponent D6
 U 1 1 5C2BA129
 P 3250 2550
@@
 $EndComp
 $Comp
-L BudKiCadComponent:LED_Cree-PLCC4 D5
+L bluetoothGame-rescue:LED_Cree-PLCC4-BudKiCadComponent D5
 U 1 1 5C2BA12F
 P 3100 5450
@@
 $EndComp
 $Comp
-L BudKiCadComponent:LED_Cree-PLCC4 D8
+L bluetoothGame-rescue:LED_Cree-PLCC4-BudKiCadComponent D8
 U 1 1 5C2BA135
 P 3800 2550
@@
 $EndComp
 $Comp
-L BudKiCadComponent:LED_Cree-PLCC4 D7
+L bluetoothGame-rescue:LED_Cree-PLCC4-BudKiCadComponent D7
 U 1 1 5C2BA13B
 P 3650 5450
@@
 	12800 7100 12800 6900
 $Comp
-L BudKiCadComponent:UM6K33NTN Q1
+L bluetoothGame-rescue:UM6K33NTN-BudKiCadComponent Q1
 U 2 1 5C29AC1A
 P 2950 3300
@@
 $EndComp
 $Comp
-L BudKiCadComponent:UM6K33NTN Q1
+L bluetoothGame-rescue:UM6K33NTN-BudKiCadComponent Q1
 U 1 1 5C29ACE0
 P 2800 6200
